File: hardware/board-v1/nexta.kicad_pcb (KiCad board)
At the start: 2 copper layers, 88.9 x 53.3 mm, 27 parts

Commit message: 4 Aruco markers, and faceplate.
Parts:
- removed the REF** at (139.8, 89.8)
- added REF**: aruco4x4-4, Aruco_Library:aruco4x4-4, F.Cu at (158.0, 89.4)
- added REF**: aruco4x4-3, Aruco_Library:aruco4x4-3, F.Cu at (120.1, 89.4)
- added REF**: MountingHole_3.2mm_M3, MountingHole:MountingHole_3.2mm_M3, F.Cu at (139.2, 89.4)
Routing:
- net Net-(A1-PadD28): track 56.8 -> 60.3 mm
- net Net-(A1-PadD27): track 63.1 -> 65.8 mm
- net Net-(A1-PadD26): track 63.3 -> 65.3 mm
- net Net-(BAR1-A-Pad10): track 15.4 -> 17.0 mm
- net Net-(BAR2-A-Pad1): track 18.8 -> 20.3 mm
- net Net-(A1-PadD25): track 69.2 -> 70.6 mm
- net Net-(A1-PadD24): track 69.2 -> 70.0 mm
- net Net-(A1-D18/TX1): track 86.1 -> 85.3 mm
- net Net-(A1-PadD30): track 50.8 -> 50.1 mm
- net Net-(A1-PadD29): track 56.8 -> 56.1 mm
- net Net-(A1-PadD31): track 48.9 -> 48.4 mm
Other:
- board text added: "Timing Board v2.0.0"
- board text removed: "Timing Board v1.1.0"
